File: PCB/TheONETXModule.sch (KiCad schematic (older format))
At the start: 4 parts, among them J1 Conn_01x05_Female

Commit message: PCB pushed to V 0.2
....created PCB for JR sized slot and already in beta testing ...PCB manufracted by AISLER
Parts:
- removed R2: 10K, Resistors_THT:R_Axial_DIN0204_L3.6mm_D1.6mm_P5.08mm_Horizontal, symbol R
- added 22uF1, 22uF2, 22uF3: CP1, Capacitors_THT:CP_Radial_Tantal_D4.5mm_P2.50mm, symbol CP1-RESCUE-TheONETXModule
- added D1, D2: LED, LEDs:LED_D3.0mm, symbol LED-RESCUE-TheONETXModule
- added D3, D4: D, Diodes_THT:D_T-1_P5.08mm_Horizontal, symbol D
- added H1: HEX_CODER_16, customs:HEX_ENCODER_16, symbol HEX_CODER_16
- added JP1: TEL_RX, customs:Jumper_SMD, symbol Jumper
- added JP2: TEL_TX, customs:Jumper_SMD, symbol Jumper
- added R2: 470, Resistors_THT:R_Axial_DIN0204_L3.6mm_D1.6mm_P5.08mm_Horizontal, symbol R-RESCUE-TheONETXModule
- added R3, R4: 1K, Resistors_THT:R_Axial_DIN0204_L3.6mm_D1.6mm_P5.08mm_Horizontal, symbol R-RESCUE-TheONETXModule
- added SW1: Bind Button, Buttons_Switches_THT:SW_PUSH_6mm, symbol SW_Push
- added T1: A7105-Hubsan, customs:A7105, symbol A7105-Hubsan
- added U1: L7805, TO_SOT_Packages_THT:TO-220-3_Horizontal, symbol L7805
- added U2: LD1117S33, TO_SOT_Packages_THT:TO-220-3_Horizontal, symbol LD1117S33TR_SOT223
- added U3: NRF24L01, customs:NRF24L01_PA, symbol NRF24L01-RESCUE-TheONETXModule
- added U4: LogicShift, customs:4Ch-LogicShift, symbol LogicShift
- A1: footprint Modules:Arduino_Nano -> Modules:Arduino_Nano_WithMountingHoles
- R1: symbol R -> R-RESCUE-TheONETXModule
Connections:
- net labels added: 3.3V, 5V, A0, A7105_CS, A7105_CS_LV, D10, D11, D12, MISO, MOSI, MOSI_LV, NRF24_CS, PB5, PPM, PPM_IN, RX_IN, SCK, SCK_LV, TX_IN, VBAT+
- wire segments 7 -> 89
- no-connect marks 0 -> 21

Commit message: ...bump
...bump
Parts:
- removed D3: D, Diodes_THT:D_T-1_P5.08mm_Horizontal, symbol D
- renumbered D4 to D1, D1 to D2, D2 to D3, U4 to U3, U3 to U4
Connections:
- wire segments 89 -> 88
Changed lines of the file:
@@
 $EndComp
 $Comp
-L LED-RESCUE-TheONETXModule D1
+L LED-RESCUE-TheONETXModule D2
 U 1 1 5A94BC0E
 P 4400 6450
-F 0 "D1" H 4400 6550 50  0000 C CNN
+F 0 "D2" H 4400 6550 50  0000 C CNN
 F 1 "LED" H 4400 6350 50  0000 C CNN
 F 2 "LEDs:LED_D3.0mm" H 4400 6450 60  0001 C CNN
@@
 $EndComp
 $Comp
-L NRF24L01-RESCUE-TheONETXModule U3
+L NRF24L01-RESCUE-TheONETXModule U4
 U 1 1 5A94D611
 P 8900 3200
-F 0 "U3" H 9200 2600 60  0000 C CNN
+F 0 "U4" H 9200 2600 60  0000 C CNN
 F 1 "NRF24L01" V 9200 3650 60  0000 C CNN
 F 2 "customs:NRF24L01_PA" H 8900 2800 60  0001 C CNN
@@
 $EndComp
 $Comp
-L GND-RESCUE-TheONETXModule #PWR01
+L GND-RESCUE-TheONETXModule #PWR6
 U 1 1 5A94DE18
 P 8050 2650
-F 0 "#PWR01" H 8050 2650 30  0001 C CNN
+F 0 "#PWR6" H 8050 2650 30  0001 C CNN
 F 1 "GND" H 8050 2580 30  0001 C CNN
 F 2 "" H 8050 2650 60  0000 C CNN
@@
 NoConn ~ 8200 2050
 $Comp
-L GND-RESCUE-TheONETXModule #PWR02
+L GND-RESCUE-TheONETXModule #PWR5
 U 1 1 5A960123
 P 7250 1550
-F 0 "#PWR02" H 7250 1550 30  0001 C CNN
+F 0 "#PWR5" H 7250 1550 30  0001 C CNN
 F 1 "GND" H 7250 1480 30  0001 C CNN
 F 2 "" H 7250 1550 60  0000 C CNN
@@
 $EndComp
 $Comp
-L GND-RESCUE-TheONETXModule #PWR03
+L GND-RESCUE-TheONETXModule #PWR3
 U 1 1 5A960420
 P 5900 6800
-F 0 "#PWR03" H 5900 6800 30  0001 C CNN
+F 0 "#PWR3" H 5900 6800 30  0001 C CNN
 F 1 "GND" H 5900 6730 30  0001 C CNN
 F 2 "" H 5900 6800 60  0000 C CNN
@@
 $EndComp
 $Comp
-L LogicShift U4
+L LogicShift U3
 U 1 1 5A986367
 P 5950 1900
-F 0 "U4" H 6200 1900 60  0000 C CNN
+F 0 "U3" H 6200 1900 60  0000 C CNN
 F 1 "LogicShift" H 5850 1900 60  0000 C CNN
 F 2 "customs:4Ch-LogicShift" H 5950 1900 60  0001 C CNN
@@
 5V
 $Comp
-L GND-RESCUE-TheONETXModule #PWR04
+L GND-RESCUE-TheONETXModule #PWR2
 U 1 1 5A9886D2
 P 5050 1950
-F 0 "#PWR04" H 5050 1950 30  0001 C CNN
+F 0 "#PWR2" H 5050 1950 30  0001 C CNN
 F 1 "GND" H 5050 1880 30  0001 C CNN
 F 2 "" H 5050 1950 60  0000 C CNN
@@
 $EndComp
 $Comp
-L GND-RESCUE-TheONETXModule #PWR05
+L GND-RESCUE-TheONETXModule #PWR4
 U 1 1 5A988B4E
 P 6950 1950
-F 0 "#PWR05" H 6950 1950 30  0001 C CNN
+F 0 "#PWR4" H 6950 1950 30  0001 C CNN
 F 1 "GND" H 6950 1880 30  0001 C CNN
 F 2 "" H 6950 1950 60  0000 C CNN
@@
 A0
 $Comp
-L GND-RESCUE-TheONETXModule #PWR06
+L GND-RESCUE-TheONETXModule #PWR8
 U 1 1 5A9B4DCF
 P 9700 5400
-F 0 "#PWR06" H 9700 5400 30  0001 C CNN
+F 0 "#PWR8" H 9700 5400 30  0001 C CNN
 F 1 "GND" H 9700 5330 30  0001 C CNN
 F 2 "" H 9700 5400 60  0000 C CNN
@@
 D12
 $Comp
-L LED-RESCUE-TheONETXModule D2
+L LED-RESCUE-TheONETXModule D3
 U 1 1 5A9B5BF8
 P 4800 3100
-F 0 "D2" H 4800 3200 50  0001 C CNN
+F 0 "D3" H 4800 3200 50  0001 C CNN
 F 1 "LED" H 4800 3000 50  0000 C CNN
 F 2 "LEDs:LED_D3.0mm" H 4800 3100 60  0001 C CNN
@@
 $EndComp
 $Comp
-L GND-RESCUE-TheONETXModule #PWR07
+L GND-RESCUE-TheONETXModule #PWR1
 U 1 1 5A9B5D4A
 P 3800 3550
-F 0 "#PWR07" H 3800 3550 30  0001 C CNN
+F 0 "#PWR1" H 3800 3550 30  0001 C CNN
 F 1 "GND" H 3800 3480 30  0001 C CNN
 F 2 "" H 3800 3550 60  0000 C CNN
@@
 D10
 $Comp
-L GND-RESCUE-TheONETXModule #PWR08
+L GND-RESCUE-TheONETXModule #PWR7
 U 1 1 5A9B81B5
 P 8450 5400
-F 0 "#PWR08" H 8450 5400 30  0001 C CNN
+F 0 "#PWR7" H 8450 5400 30  0001 C CNN
 F 1 "GND" H 8450 5330 30  0001 C CNN
 F 2 "" H 8450 5400 60  0000 C CNN
@@
 	-1   0    0    -1
 $EndComp
-$Comp
-L D D3
-U 1 1 5AB17D63
-P 2400 5300
-F 0 "D3" H 2250 5350 50  0000 C CNN
-F 1 "D" H 2500 5350 50  0000 C CNN
-F 2 "Diodes_THT:D_T-1_P5.08mm_Horizontal" H 2400 5300 50  0001 C CNN
-F 3 "" H 2400 5300 50  0001 C CNN
-	1    2400 5300
-	-1   0    0    1
-$EndComp
-Wire Wire Line
-	2250 5300 2200 5300
-$Comp
-L D D4
+Wire Wire Line
+	2200 5300 5900 5300
+$Comp
+L D D1
 U 1 1 5AB1806F
 P 2400 5500
-F 0 "D4" H 2250 5550 50  0000 C CNN
+F 0 "D1" H 2250 5550 50  0000 C CNN
 F 1 "D" H 2500 5550 50  0000 C CNN
 F 2 "Diodes_THT:D_T-1_P5.08mm_Horizontal" H 2400 5500 50  0001 C CNN
@@
 $EndComp
 Wire Wire Line
-	2550 5300 5900 5300
-Wire Wire Line
 	2700 5100 2700 5300

Commit message: ...
Parts:
- removed T1: A7105-Hubsan, customs:A7105, symbol A7105-Hubsan
- added R5: 10K, Resistors_THT:R_Axial_DIN0204_L3.6mm_D1.6mm_P5.08mm_Horizontal, symbol TheONETXModule-rescue:R-RESCUE-TheONETXModule
- added U5: A7105, customs:A7106, symbol TheONETXModule-rescue:A7105
- 22uF1, 22uF2, 22uF3: footprint Capacitors_THT:CP_Radial_Tantal_D4.5mm_P2.50mm -> Capacitors_THT:CP_Radial_D5.0mm_P2.50mm; symbol CP1-RESCUE-TheONETXModule -> TheONETXModule-rescue:CP1-RESCUE-TheONETXModule
- A1: symbol Arduino_Nano_v3.x -> TheONETXModule-rescue:Arduino_Nano_v3.x-modules
- D1: footprint Diodes_THT:D_T-1_P5.08mm_Horizontal -> Diodes_THT:D_5W_P10.16mm_Horizontal; symbol D -> Device:D
- D2, D3: symbol LED-RESCUE-TheONETXModule -> TheONETXModule-rescue:LED-RESCUE-TheONETXModule
- H1: symbol HEX_CODER_16 -> TheONETXParts:HEX_CODER_16
- J1: symbol Conn_01x05_Female -> TheONETXParts:Conn_01x05_Female
- JP1, JP2: symbol Jumper -> Device:Jumper
- R1, R2, R3, R4: symbol R-RESCUE-TheONETXModule -> TheONETXModule-rescue:R-RESCUE-TheONETXModule
- SW1: symbol SW_Push -> TheONETXModule-rescue:SW_Push-switches
- U1: footprint TO_SOT_Packages_THT:TO-220-3_Horizontal -> TO_SOT_Packages_SMD:SOT-223; symbol L7805 -> TheONETXParts:L7805
- U2: footprint TO_SOT_Packages_THT:TO-220-3_Horizontal -> TO_SOT_Packages_SMD:SOT-223; symbol LD1117S33TR_SOT223 -> TheONETXParts:LD1117S33TR_SOT223
- U3: symbol LogicShift -> TheONETXParts:LogicShift
- U4: symbol NRF24L01-RESCUE-TheONETXModule -> TheONETXModule-rescue:NRF24L01-RESCUE-TheONETXModule
Connections:
- net labels added: 5V_int
- wire segments 88 -> 116
- no-connect marks 21 -> 17
Other:
- moved on the sheet: 22uF1, R3
